File: lpc1754/lpc1754_board.sch (KiCad schematic (older format))
At the start: 34 parts, among them IC1 LPC175X, J1 USB, SW1 SWITCH_PUSHBUTTON, U3 CONN_CORTEX_DEBUG, X1 CRYSTAL_MINI, X2 CRYSTAL_MINI

Commit message: Drills de 1mm con vias de 1.6mm
Signed-off-by: Martin Ribelotta <martinribelotta@gmail.com>
Parts:
- C1: value C_MINI -> 0.1uF
- C10, C11, C12, C331, C6, C7, C8, C9: value C_MINI -> 0.1uf
- C2, C3, C4, C5: value C_MINI -> 18pf
- C332, C_VIN1: value CP_TANTALUM_MINI -> 10uf
- R1, R2, R3, R7: value R_MINI -> 10K
- R4, R5: value R_MINI -> 33R
- R6: value R_MINI -> 1K5
- R8: value R_MINI -> 1K
- X1: value CRYSTAL_MINI -> 32.768kHz
- X2: value CRYSTAL_MINI -> 25Mhz
Changed lines of the file:
@@
-EESchema Schematic File Version 2  date sáb 09 abr 2011 22:18:57 ART
+EESchema Schematic File Version 2  date 12/04/2011 09:37:18 p.m.
 LIBS:power
 LIBS:device
@@
 Sheet 1 1
 Title ""
-Date "10 apr 2011"
+Date "13 apr 2011"
 Rev ""
 Comp ""
@@
 P 10450 1450
 F 0 "R8" H 10380 1500 25  0000 C CNN
-F 1 "R_MINI" H 10520 1500 20  0000 C CNN
+F 1 "1K" H 10520 1500 20  0000 C CNN
 	1    10450 1450
 	0    -1   -1   0
@@
 P 8550 5800
 F 0 "R7" H 8480 5850 25  0000 C CNN
-F 1 "R_MINI" H 8620 5850 20  0000 C CNN
+F 1 "10K" H 8620 5850 20  0000 C CNN
 	1    8550 5800
 	-1   0    0    1
@@
 P 8650 1450
 F 0 "C_VIN1" V 8600 1490 30  0000 C CNN
-F 1 "CP_TANTALUM_MINI" V 8700 1520 25  0000 C CNN
+F 1 "10uf" V 8700 1520 25  0000 C CNN
 	1    8650 1450
 	0    1    1    0
@@
 P 10100 1450
 F 0 "C332" V 10050 1490 30  0000 C CNN
-F 1 "CP_TANTALUM_MINI" V 10150 1520 25  0000 C CNN
+F 1 "10uf" V 10150 1520 25  0000 C CNN
 	1    10100 1450
 	0    1    1    0
@@
 P 9650 1450
 F 0 "C331" V 9600 1490 30  0000 C CNN
-F 1 "C_MINI" V 9700 1520 25  0000 C CNN
+F 1 "0.1uf" V 9700 1520 25  0000 C CNN
 	1    9650 1450
 	0    1    1    0
@@
 P 3650 3300
 F 0 "R6" H 3580 3350 25  0000 C CNN
-F 1 "R_MINI" H 3720 3350 20  0000 C CNN
+F 1 "1K5" H 3720 3350 20  0000 C CNN
 	1    3650 3300
 	-1   0    0    1
@@
 P 3650 3500
 F 0 "R4" H 3580 3550 25  0000 C CNN
-F 1 "R_MINI" H 3720 3550 20  0000 C CNN
+F 1 "33R" H 3720 3550 20  0000 C CNN
 	1    3650 3500
 	-1   0    0    1
@@
 P 3650 3400
 F 0 "R5" H 3580 3450 25  0000 C CNN
-F 1 "R_MINI" H 3720 3450 20  0000 C CNN
+F 1 "33R" H 3720 3450 20  0000 C CNN
 	1    3650 3400
 	-1   0    0    1
@@
 P 3650 3800
 F 0 "R3" H 3580 3850 25  0000 C CNN
-F 1 "R_MINI" H 3720 3850 20  0000 C CNN
+F 1 "10K" H 3720 3850 20  0000 C CNN
 	1    3650 3800
 	-1   0    0    1
@@
 P 3650 3650
 F 0 "R2" H 3580 3700 25  0000 C CNN
-F 1 "R_MINI" H 3720 3700 20  0000 C CNN
+F 1 "10K" H 3720 3700 20  0000 C CNN
 	1    3650 3650
 	-1   0    0    1
@@
 P 3900 2250
 F 0 "X2" H 3900 2150 35  0000 C CNN
-F 1 "CRYSTAL_MINI" H 3900 2350 25  0000 C CNN
+F 1 "25Mhz" H 3900 2350 25  0000 C CNN
 	1    3900 2250
 	1    0    0    -1
@@
 U 1 1 4D9FBF16
 P 2050 3100
-F 0 "C1" V 2000 3140 30  0000 C CNN
-F 1 "C_MINI" V 2100 3170 25  0000 C CNN
+F 0 "C1" H 1950 3150 30  0000 C CNN
+F 1 "0.1uF" H 2100 3170 25  0000 C CNN
 	1    2050 3100
 	-1   0    0    1
@@
 P 2600 2950
 F 0 "R1" H 2530 3000 25  0000 C CNN
-F 1 "R_MINI" H 2670 3000 20  0000 C CNN
+F 1 "10K" H 2670 3000 20  0000 C CNN
 	1    2600 2950
 	0    1    1    0
@@
 P 4100 1800
 F 0 "C5" V 4050 1840 30  0000 C CNN
-F 1 "C_MINI" V 4150 1870 25  0000 C CNN
+F 1 "18pf" V 4150 1870 25  0000 C CNN
 	1    4100 1800
 	0    1    1    0
@@
 P 3700 1800
 F 0 "C4" V 3650 1840 30  0000 C CNN
-F 1 "C_MINI" V 3750 1870 25  0000 C CNN
+F 1 "18pf" V 3750 1870 25  0000 C CNN
 	1    3700 1800
 	0    1    1    0
@@
 P 3300 1800
 F 0 "C3" V 3250 1840 30  0000 C CNN
-F 1 "C_MINI" V 3350 1870 25  0000 C CNN
+F 1 "18pf" V 3350 1870 25  0000 C CNN
 	1    3300 1800
 	0    1    1    0
@@
 P 2900 1800
 F 0 "C2" V 2850 1840 30  0000 C CNN
-F 1 "C_MINI" V 2950 1870 25  0000 C CNN
+F 1 "18pf" V 2950 1870 25  0000 C CNN
 	1    2900 1800
 	0    1    1    0
@@
 P 3100 2250
 F 0 "X1" H 3100 2150 35  0000 C CNN
-F 1 "CRYSTAL_MINI" H 3100 2350 25  0000 C CNN
+F 1 "32.768kHz" H 3100 2350 25  0000 C CNN
 	1    3100 2250
 	1    0    0    -1
@@
 P 6550 1950
 F 0 "C12" V 6500 1990 30  0000 C CNN
-F 1 "C_MINI" V 6600 2020 25  0000 C CNN
+F 1 "0.1uf" V 6600 2020 25  0000 C CNN
 	1    6550 1950
 	-1   0    0    1
@@
 P 6550 1750
 F 0 "C11" V 6500 1790 30  0000 C CNN
-F 1 "C_MINI" V 6600 1820 25  0000 C CNN
+F 1 "0.1uf" V 6600 1820 25  0000 C CNN
 	1    6550 1750
 	-1   0    0    1
@@
 P 6550 1550
 F 0 "C10" V 6500 1590 30  0000 C CNN
-F 1 "C_MINI" V 6600 1620 25  0000 C CNN
+F 1 "0.1uf" V 6600 1620 25  0000 C CNN
 	1    6550 1550
 	-1   0    0    1
@@
 P 5400 1550
 F 0 "C6" V 5350 1590 30  0000 C CNN
-F 1 "C_MINI" V 5450 1620 25  0000 C CNN
+F 1 "0.1uf" V 5450 1620 25  0000 C CNN
 	1    5400 1550
 	1    0    0    -1
@@
 P 5400 1750
 F 0 "C7" V 5350 1790 30  0000 C CNN
-F 1 "C_MINI" V 5450 1820 25  0000 C CNN
+F 1 "0.1uf" V 5450 1820 25  0000 C CNN
 	1    5400 1750
 	1    0    0    -1
@@
 P 5400 1950
 F 0 "C8" V 5350 1990 30  0000 C CNN
-F 1 "C_MINI" V 5450 2020 25  0000 C CNN
+F 1 "0.1uf" V 5450 2020 25  0000 C CNN
 	1    5400 1950
 	1    0    0    -1
@@
 P 5400 2150
 F 0 "C9" V 5350 2190 30  0000 C CNN
-F 1 "C_MINI" V 5450 2220 25  0000 C CNN
+F 1 "0.1uf" V 5450 2220 25  0000 C CNN
 	1    5400 2150
 	1    0    0    -1

Commit message: Conector JTAG corregido, planos de masa retirados del conector de los pines
Signed-off-by: Martin Ribelotta <martinribelotta@gmail.com>
Parts:
- removed U3: CONN_CORTEX_DEBUG, symbol CONN_CORTEX_DEBUG
- added P1: CONN_4X2, symbol CONN_4X2
Connections:
- net labels added: TCK, TDI, TDO, TMS, TRST
- wire segments 174 -> 164
Changed lines of the file:
@@
-EESchema Schematic File Version 2  date 12/04/2011 09:37:18 p.m.
+EESchema Schematic File Version 2  date 12/04/2011 10:32:49 p.m.
 LIBS:power
 LIBS:device
@@
 Comment4 ""
 $EndDescr
+Text Label 3800 5950 0    60   ~ 0
+TCK
+Text Label 3800 5850 0    60   ~ 0
+TRST
+Text Label 3800 5750 0    60   ~ 0
+TMS
+Text Label 3800 5650 0    60   ~ 0
+TDI
+Text Label 3800 5550 0    60   ~ 0
+TDO
+Wire Wire Line
+	4300 5950 3800 5950
+Wire Wire Line
+	4300 5750 3800 5750
+Wire Wire Line
+	4300 5550 3800 5550
+Wire Wire Line
+	2550 4650 2850 4650
+Wire Wire Line
+	2700 5000 2700 4550
+Wire Wire Line
+	1750 4750 1350 4750
+Wire Wire Line
+	1600 4450 1600 4550
+Wire Wire Line
+	1600 4550 1750 4550
 Connection ~ 9700 4600
 Wire Wire Line
@@
 Wire Wire Line
 	4250 6250 4300 6250
-Wire Wire Line
-	4300 5850 3350 5850
-Wire Wire Line
-	3350 5850 3350 5900
-Wire Wire Line
-	3350 5900 3000 5900
-Wire Wire Line
-	3000 5900 3000 5950
-Wire Wire Line
-	3000 5950 2650 5950
-Wire Wire Line
-	1550 6200 1550 5650
-Wire Wire Line
-	1650 5550 1550 5550
-Connection ~ 1550 5950
-Wire Wire Line
-	1650 5950 1550 5950
-Wire Wire Line
-	2650 5650 3050 5650
-Wire Wire Line
-	3050 5650 3050 5950
-Wire Wire Line
-	3050 5950 4300 5950
-Wire Wire Line
-	2650 5850 3300 5850
-Wire Wire Line
-	3300 5850 3300 5650
 Wire Wire Line
 	5600 6900 5600 6450
@@
 Connection ~ 5600 6650
 Wire Wire Line
-	4300 5750 3200 5750
-Wire Wire Line
-	3200 5750 3200 5550
-Wire Wire Line
-	3200 5550 2650 5550
-Wire Wire Line
-	4300 5550 3250 5550
-Wire Wire Line
-	3250 5550 3250 5650
-Wire Wire Line
-	3250 5650 3150 5650
-Wire Wire Line
-	3150 5650 3150 5750
-Wire Wire Line
-	3150 5750 2650 5750
-Wire Wire Line
-	1550 5650 1650 5650
-Wire Wire Line
-	1650 5750 1550 5750
-Connection ~ 1550 5750
-Wire Wire Line
-	1550 5550 1550 5250
-Wire Wire Line
-	3300 5650 4300 5650
-Wire Wire Line
 	4300 6150 4050 6150
 Wire Wire Line
@@
 	9750 7100 9750 7000
 Connection ~ 9750 7000
+Wire Wire Line
+	2700 4550 2550 4550
+Wire Wire Line
+	1750 4650 1350 4650
+Wire Wire Line
+	1750 4850 1350 4850
+Wire Wire Line
+	2550 4850 2700 4850
+Connection ~ 2700 4850
+Wire Wire Line
+	2550 4750 2850 4750
+Wire Wire Line
+	4300 5650 3800 5650
+Wire Wire Line
+	4300 5850 3800 5850
+Text Label 2850 4650 0    60   ~ 0
+TDO
+Text Label 2850 4750 0    60   ~ 0
+TMS
+Text Label 1350 4850 0    60   ~ 0
+TRST
+Text Label 1350 4750 0    60   ~ 0
+TDI
+Text Label 1350 4650 0    60   ~ 0
+TCK
+$Comp
+L CONN_4X2 P1
+U 1 1 4DA4F950
+P 2150 4700
+F 0 "P1" H 2150 4950 50  0000 C CNN
+F 1 "CONN_4X2" V 2150 4700 40  0000 C CNN
+	1    2150 4700
+	1    0    0    -1
+$EndComp
 $Comp
 L +3.3V #PWR01
@@
 $EndComp
 $Comp
-L GND #PWR03
+L GND #PWR02
 U 1 1 4DA104B4
 P 9600 4650
-F 0 "#PWR03" H 9600 4650 30  0001 C CNN
+F 0 "#PWR02" H 9600 4650 30  0001 C CNN
 F 1 "GND" H 9600 4580 30  0001 C CNN
 	1    9600 4650
@@
 $EndComp
 $Comp
-L VBUS #PWR05
+L VBUS #PWR03
 U 1 1 4DA0FD20
 P 8250 1050
-F 0 "#PWR05" H 8250 1150 30  0001 C CNN
+F 0 "#PWR03" H 8250 1150 30  0001 C CNN
 F 1 "VBUS" H 8250 1150 30  0000 C CNN
 	1    8250 1050
@@
 $EndComp
 $Comp
-L +3.3V #PWR06
+L +3.3V #PWR04
 U 1 1 4DA083BC
 P 9950 1150
-F 0 "#PWR06" H 9950 1110 30  0001 C CNN
+F 0 "#PWR04" H 9950 1110 30  0001 C CNN
 F 1 "+3.3V" H 9950 1260 30  0000 C CNN
 	1    9950 1150
@@
 $EndComp
 $Comp
-L +3.3V #PWR07
+L +3.3V #PWR05
 U 1 1 4DA08361
 P 8900 5800
-F 0 "#PWR07" H 8900 5760 30  0001 C CNN
+F 0 "#PWR05" H 8900 5760 30  0001 C CNN
 F 1 "+3.3V" H 8900 5910 30  0000 C CNN
 	1    8900 5800
@@
 $EndComp
 $Comp
-L GND #PWR08
+L GND #PWR06
 U 1 1 4DA08354
 P 8350 6250
-F 0 "#PWR08" H 8350 6250 30  0001 C CNN
+F 0 "#PWR06" H 8350 6250 30  0001 C CNN
 F 1 "GND" H 8350 6180 30  0001 C CNN
 	1    8350 6250
@@
 $EndComp
 $Comp
-L GND #PWR09
+L GND #PWR07
 U 1 1 4D9FD592
 P 9050 1800
-F 0 "#PWR09" H 9050 1800 30  0001 C CNN
+F 0 "#PWR07" H 9050 1800 30  0001 C CNN
 F 1 "GND" H 9050 1730 30  0001 C CNN
 	1    9050 1800
@@
 $EndComp
 $Comp
-L +3.3V #PWR010
+L +3.3V #PWR08
 U 1 1 4D9FCFA7
 P 3900 3300
-F 0 "#PWR010" H 3900 3260 30  0001 C CNN
+F 0 "#PWR08" H 3900 3260 30  0001 C CNN
 F 1 "+3.3V" H 3900 3410 30  0000 C CNN
 	1    3900 3300
@@
 $EndComp
 $Comp
-L GND #PWR011
+L GND #PWR09
 U 1 1 4D9FCBEB
 P 3400 3800
-F 0 "#PWR011" H 3400 3800 30  0001 C CNN
+F 0 "#PWR09" H 3400 3800 30  0001 C CNN
 F 1 "GND" H 3400 3730 30  0001 C CNN
 	1    3400 3800
@@
 $EndComp
 $Comp
-L VBUS #PWR012
+L VBUS #PWR010
 U 1 1 4D9FCBD5
 P 3450 3650
-F 0 "#PWR012" H 3450 3750 30  0001 C CNN
+F 0 "#PWR010" H 3450 3750 30  0001 C CNN
 F 1 "VBUS" H 3450 3750 30  0000 C CNN
 	1    3450 3650
@@
 $EndComp
 $Comp
-L VBUS #PWR013
+L VBUS #PWR011
 U 1 1 4D9FCBD0
 P 1050 3800
-F 0 "#PWR013" H 1050 3900 30  0001 C CNN
+F 0 "#PWR011" H 1050 3900 30  0001 C CNN
 F 1 "VBUS" H 1050 3900 30  0000 C CNN
 	1    1050 3800
@@
 $EndComp
 $Comp
-L GND #PWR014
+L GND #PWR012
 U 1 1 4D9FCBA6
 P 750 3500
-F 0 "#PWR014" H 750 3500 30  0001 C CNN
+F 0 "#PWR012" H 750 3500 30  0001 C CNN
 F 1 "GND" H 750 3430 30  0001 C CNN
 	1    750  3500
@@
 $EndComp
 $Comp
-L GND #PWR015
+L GND #PWR013
 U 1 1 4D9FC66B
 P 4250 6350
-F 0 "#PWR015" H 4250 6350 30  0001 C CNN
+F 0 "#PWR013" H 4250 6350 30  0001 C CNN
 F 1 "GND" H 4250 6280 30  0001 C CNN
 	1    4250 6350
@@
 $EndComp
 $Comp
-L +3.3V #PWR016
+L +3.3V #PWR014
 U 1 1 4D9FC667
 P 4050 6150
-F 0 "#PWR016" H 4050 6110 30  0001 C CNN
+F 0 "#PWR014" H 4050 6110 30  0001 C CNN
 F 1 "+3.3V" H 4050 6260 30  0000 C CNN
 	1    4050 6150
@@
 $EndComp
 $Comp
-L +3.3V #PWR017
+L +3.3V #PWR015
 U 1 1 4D9FC639
-P 1550 5250
-F 0 "#PWR017" H 1550 5210 30  0001 C CNN
-F 1 "+3.3V" H 1550 5360 30  0000 C CNN
-	1    1550 5250
-	1    0    0    -1
-$EndComp
-$Comp
-L GND #PWR018
+P 1600 4450
+F 0 "#PWR015" H 1600 4410 30  0001 C CNN
+F 1 "+3.3V" H 1600 4560 30  0000 C CNN
+	1    1600 4450
+	1    0    0    -1
+$EndComp
+$Comp
+L GND #PWR016
 U 1 1 4D9FC633
-P 1550 6200
-F 0 "#PWR018" H 1550 6200 30  0001 C CNN
-F 1 "GND" H 1550 6130 30  0001 C CNN
-	1    1550 6200
-	1    0    0    -1
-$EndComp
-$Comp
-L CONN_CORTEX_DEBUG U3
-U 1 1 4D9FC5A1
-P 2150 5750
-F 0 "U3" H 2150 5450 50  0000 C CNN
-F 1 "CONN_CORTEX_DEBUG" H 2150 6050 35  0000 C CNN
-	1    2150 5750
+P 2700 5000
+F 0 "#PWR016" H 2700 5000 30  0001 C CNN
+F 1 "GND" H 2700 4930 30  0001 C CNN
+	1    2700 5000
 	1    0    0    -1
 $EndComp
@@
 $EndComp
 $Comp
-L GND #PWR019
+L GND #PWR017
 U 1 1 4D9FBFA4
 P 5600 6900
-F 0 "#PWR019" H 5600 6900 30  0001 C CNN
+F 0 "#PWR017" H 5600 6900 30  0001 C CNN
 F 1 "GND" H 5600 6830 30  0001 C CNN
 	1    5600 6900
@@
 $EndComp
 $Comp
-L +3.3V #PWR020
+L +3.3V #PWR018
 U 1 1 4D9FBF87
 P 2600 2800
-F 0 "#PWR020" H 2600 2760 30  0001 C CNN
+F 0 "#PWR018" H 2600 2760 30  0001 C CNN
 F 1 "+3.3V" H 2600 2910 30  0000 C CNN
 	1    2600 2800
@@
 $EndComp
 $Comp
-L GND #PWR021
+L GND #PWR019
 U 1 1 4D9FBF37
 P 1800 3100
-F 0 "#PWR021" H 1800 3100 30  0001 C CNN
+F 0 "#PWR019" H 1800 3100 30  0001 C CNN
 F 1 "GND" H 1800 3030 30  0001 C CNN
 	1    1800 3100
@@
 $EndComp
 $Comp
-L GND #PWR022
+L GND #PWR020
 U 1 1 4D9FBEF0
 P 3500 1800
-F 0 "#PWR022" H 3500 1800 30  0001 C CNN
+F 0 "#PWR020" H 3500 1800 30  0001 C CNN
 F 1 "GND" H 3500 1730 30  0001 C CNN
 	1    3500 1800
@@
 $EndComp
 $Comp
-L GND #PWR023
+L GND #PWR021
 U 1 1 4D9FBBA7
 P 6900 2050
-F 0 "#PWR023" H 6900 2050 30  0001 C CNN
+F 0 "#PWR021" H 6900 2050 30  0001 C CNN
 F 1 "GND" H 6900 1980 30  0001 C CNN
 	1    6900 2050
@@
 $EndComp
 $Comp
-L +3.3V #PWR024
+L +3.3V #PWR022
 U 1 1 4D9FBB67
 P 5600 1300
-F 0 "#PWR024" H 5600 1260 30  0001 C CNN
+F 0 "#PWR022" H 5600 1260 30  0001 C CNN
 F 1 "+3.3V" H 5600 1410 30  0000 C CNN
 	1    5600 1300
@@
 $EndComp
 $Comp
-L GND #PWR025
+L GND #PWR023
 U 1 1 4D9FBB51
 P 5050 1750
-F 0 "#PWR025" H 5050 1750 30  0001 C CNN
+F 0 "#PWR023" H 5050 1750 30  0001 C CNN
 F 1 "GND" H 5050 1680 30  0001 C CNN
 	1    5050 1750

Commit message: Agregado USB-HOST en placa LPC1754. DRC en esquematico y PCB
Parts:
- added J_HOST1: USB_2, symbol USB_2
Connections:
- net labels added: +5V
- wire segments 164 -> 172
- no-connect marks 0 -> 7
Other:
- moved on the sheet: P_IO1, R4, R5, R6

Commit message: lpc1754: Corregido el conector PWR_JACK, LEDs de power y proposito general. Cambios en las pistas del impreso y GERBERS actualizados
Signed-off-by: Martin Ribelotta <martinribelotta@gmail.com>
Parts:
- added LED1, LED2: LED, symbol LED
- added R10, R9: 10K, symbol R_MINI
Connections:
- wire segments 172 -> 181
- no-connect marks 7 -> 6
Changed lines of the file:
@@
-EESchema Schematic File Version 2  date sáb 16 abr 2011 13:00:25 ART
+EESchema Schematic File Version 2  date 28/04/2011 12:44:41 p.m.
 LIBS:power
 LIBS:device
@@
 Sheet 1 1
 Title ""
-Date "16 apr 2011"
+Date "28 apr 2011"
 Rev ""
 Comp ""
@@
 Comment4 ""
 $EndDescr
-$Comp
-L +5V #PWR01
-U 1 1 4DA9B739
-P 8350 1450
-F 0 "#PWR01" H 8350 1540 20  0001 C CNN
-F 1 "+5V" H 8350 1540 30  0000 C CNN
-	1    8350 1450
-	0    1    1    0
-$EndComp
-Wire Wire Line
-	8350 1450 8000 1450
-Connection ~ 8250 1450
+Wire Wire Line
+	10350 750  10550 750
+Wire Wire Line
+	10550 750  10550 900
+Wire Wire Line
+	1250 5850 1400 5850
+Wire Wire Line
+	7650 6250 7500 6250
+Connection ~ 8050 1350
+Wire Wire Line
+	8250 1350 8000 1350
 Connection ~ 2550 3500
 Wire Wire Line
@@
 Wire Wire Line
 	7500 6000 7900 6000
-Wire Wire Line
-	8100 1550 8100 1350
-Wire Wire Line
-	8100 1350 8000 1350
 Connection ~ 9950 1250
 Wire Wire Line
@@
 Wire Wire Line
 	8250 1550 8000 1550
-Connection ~ 8100 1550
 Wire Wire Line
 	4300 4150 3850 4150
@@
 Wire Wire Line
 	7500 2850 7900 2850
-Wire Wire Line
-	8250 1450 8250 1350
 Wire Wire Line
 	9000 5000 9150 5000
@@
 	2650 4050 2650 3400
 Connection ~ 2650 3400
+Wire Wire Line
+	8050 1350 8050 1050
+Wire Wire Line
+	8000 1450 8050 1450
+Wire Wire Line
+	8050 1450 8050 1550
+Connection ~ 8050 1550
+Wire Wire Line
+	900  5850 1050 5850
+Wire Wire Line
+	1800 5850 1900 5850
+Wire Wire Line
+	1900 5850 1900 5600
+Wire Wire Line
+	9450 750  9600 750
+Wire Wire Line
+	9800 750  9950 750
+$Comp
+L GND #PWR01
+U 1 1 4DB98A0C
+P 10550 900
+F 0 "#PWR01" H 10550 900 30  0001 C CNN
+F 1 "GND" H 10550 830 30  0001 C CNN
+	1    10550 900
+	1    0    0    -1
+$EndComp
+$Comp
+L LED LED2
+U 1 1 4DB98A0B
+P 10150 750
+F 0 "LED2" H 10150 850 50  0000 C CNN
+F 1 "LED" H 10150 650 50  0000 C CNN
+	1    10150 750
+	1    0    0    -1
+$EndComp
+$Comp
+L R_MINI R10
+U 1 1 4DB98A0A
+P 9700 750
+F 0 "R10" H 9630 800 25  0000 C CNN
+F 1 "10K" H 9770 800 20  0000 C CNN
+	1    9700 750
+	-1   0    0    1
+$EndComp
+$Comp
+L +3.3V #PWR02
+U 1 1 4DB98A09
+P 9450 750
+F 0 "#PWR02" H 9450 710 30  0001 C CNN
+F 1 "+3.3V" H 9450 860 30  0000 C CNN
+	1    9450 750
+	0    -1   -1   0
+$EndComp
+$Comp
+L +3.3V #PWR03
+U 1 1 4DB989D6
+P 900 5850
+F 0 "#PWR03" H 900 5810 30  0001 C CNN
+F 1 "+3.3V" H 900 5960 30  0000 C CNN
+	1    900  5850
+	0    -1   -1   0
+$EndComp
+$Comp
+L R_MINI R9
+U 1 1 4DB989D1
+P 1150 5850
+F 0 "R9" H 1080 5900 25  0000 C CNN
+F 1 "10K" H 1220 5900 20  0000 C CNN
+	1    1150 5850
+	-1   0    0    1
+$EndComp
+$Comp
+L LED LED1
+U 1 1 4DB989BC
+P 1600 5850
+F 0 "LED1" H 1600 5950 50  0000 C CNN
+F 1 "LED" H 1600 5750 50  0000 C CNN
+	1    1600 5850
+	1    0    0    -1
+$EndComp
+Text Label 1900 5600 0    60   ~ 0
+P1.18
+$Comp
+L +3.3V #PWR04
+U 1 1 4DB980C2
+P 7650 6250
+F 0 "#PWR04" H 7650 6210 30  0001 C CNN
+F 1 "+3.3V" H 7650 6360 30  0000 C CNN
+	1    7650 6250
+	0    1    1    0
+$EndComp
+$Comp
+L +5V #PWR05
+U 1 1 4DA9B739
+P 8050 1050
+F 0 "#PWR05" H 8050 1140 20  0001 C CNN
+F 1 "+5V" H 8050 1140 30  0000 C CNN
+	1    8050 1050
+	1    0    0    -1
+$EndComp
 NoConn ~ 7500 4800
 NoConn ~ 4300 3200
@@
 NoConn ~ 850  3600
 NoConn ~ 1600 3600
-NoConn ~ 7500 6250
-$Comp
-L GND #PWR02
+$Comp
+L GND #PWR06
 U 1 1 4DA9B271
 P 2400 4300
-F 0 "#PWR02" H 2400 4300 30  0001 C CNN
+F 0 "#PWR06" H 2400 4300 30  0001 C CNN
 F 1 "GND" H 2400 4230 30  0001 C CNN
 	1    2400 4300
@@
 $EndComp
 $Comp
-L +5V #PWR03
+L +5V #PWR07
 U 1 1 4DA9B269
 P 2400 3750
-F 0 "#PWR03" H 2400 3840 20  0001 C CNN
+F 0 "#PWR07" H 2400 3840 20  0001 C CNN
 F 1 "+5V" H 2400 3840 30  0000 C CNN
 	1    2400 3750
@@
 $EndComp
 $Comp
-L +3.3V #PWR04
+L +3.3V #PWR08
 U 1 1 4DA104BC
 P 9000 5000
-F 0 "#PWR04" H 9000 4960 30  0001 C CNN
+F 0 "#PWR08" H 9000 4960 30  0001 C CNN
 F 1 "+3.3V" H 9000 5110 30  0000 C CNN
 	1    9000 5000
@@
 $EndComp
 $Comp
-L GND #PWR05
+L GND #PWR09
 U 1 1 4DA104B4
 P 8950 2650
-F 0 "#PWR05" H 8950 2650 30  0001 C CNN
+F 0 "#PWR09" H 8950 2650 30  0001 C CNN
 F 1 "GND" H 8950 2580 30  0001 C CNN
 	1    8950 2650
@@
 $EndComp
 $Comp
-L VBUS #PWR06
+L VBUS #PWR010
 U 1 1 4DA0FD20
 P 8250 1050
-F 0 "#PWR06" H 8250 1150 30  0001 C CNN
+F 0 "#PWR010" H 8250 1150 30  0001 C CNN
 F 1 "VBUS" H 8250 1150 30  0000 C CNN
 	1    8250 1050
@@
 $EndComp
 $Comp
-L +3.3V #PWR07
+L +3.3V #PWR011
 U 1 1 4DA083BC
 P 9950 1150
-F 0 "#PWR07" H 9950 1110 30  0001 C CNN
+F 0 "#PWR011" H 9950 1110 30  0001 C CNN
 F 1 "+3.3V" H 9950 1260 30  0000 C CNN
 	1    9950 1150
@@
 $EndComp
 $Comp
-L +3.3V #PWR08
+L +3.3V #PWR012
 U 1 1 4DA08361
 P 8900 5800
-F 0 "#PWR08" H 8900 5760 30  0001 C CNN
+F 0 "#PWR012" H 8900 5760 30  0001 C CNN
 F 1 "+3.3V" H 8900 5910 30  0000 C CNN
 	1    8900 5800
@@
 $EndComp
 $Comp
-L GND #PWR09
+L GND #PWR013
 U 1 1 4DA08354
 P 8350 6250
-F 0 "#PWR09" H 8350 6250 30  0001 C CNN
+F 0 "#PWR013" H 8350 6250 30  0001 C CNN
 F 1 "GND" H 8350 6180 30  0001 C CNN
 	1    8350 6250
@@
 $EndComp
 $Comp
-L GND #PWR010
+L GND #PWR014
 U 1 1 4D9FD592
 P 9050 1800
-F 0 "#PWR010" H 9050 1800 30  0001 C CNN
+F 0 "#PWR014" H 9050 1800 30  0001 C CNN
 F 1 "GND" H 9050 1730 30  0001 C CNN
 	1    9050 1800
@@
 $EndComp
 $Comp
-L +3.3V #PWR011
+L +3.3V #PWR015
 U 1 1 4D9FCFA7
 P 3950 3300
-F 0 "#PWR011" H 3950 3260 30  0001 C CNN
+F 0 "#PWR015" H 3950 3260 30  0001 C CNN
 F 1 "+3.3V" H 3950 3410 30  0000 C CNN
 	1    3950 3300
@@
 $EndComp
 $Comp
-L GND #PWR012
+L GND #PWR016
 U 1 1 4D9FCBEB
 P 3400 3800
-F 0 "#PWR012" H 3400 3800 30  0001 C CNN
+F 0 "#PWR016" H 3400 3800 30  0001 C CNN
 F 1 "GND" H 3400 3730 30  0001 C CNN
 	1    3400 3800
@@
 $EndComp
 $Comp
-L VBUS #PWR013
+L VBUS #PWR017
 U 1 1 4D9FCBD5
 P 3450 3650
-F 0 "#PWR013" H 3450 3750 30  0001 C CNN
+F 0 "#PWR017" H 3450 3750 30  0001 C CNN
 F 1 "VBUS" H 3450 3750 30  0000 C CNN
 	1    3450 3650
@@
 $EndComp
 $Comp
-L VBUS #PWR014
+L VBUS #PWR018
 U 1 1 4D9FCBD0
 P 1050 3800
-F 0 "#PWR014" H 1050 3900 30  0001 C CNN
+F 0 "#PWR018" H 1050 3900 30  0001 C CNN
 F 1 "VBUS" H 1050 3900 30  0000 C CNN
 	1    1050 3800
@@
 $EndComp
 $Comp
-L GND #PWR015
+L GND #PWR019
 U 1 1 4D9FCBA6
 P 750 3500
-F 0 "#PWR015" H 750 3500 30  0001 C CNN
+F 0 "#PWR019" H 750 3500 30  0001 C CNN
 F 1 "GND" H 750 3430 30  0001 C CNN
 	1    750  3500
@@
 $EndComp
 $Comp
-L GND #PWR016
+L GND #PWR020
 U 1 1 4D9FC66B
 P 4250 6350
-F 0 "#PWR016" H 4250 6350 30  0001 C CNN
+F 0 "#PWR020" H 4250 6350 30  0001 C CNN
 F 1 "GND" H 4250 6280 30  0001 C CNN
 	1    4250 6350
@@
 $EndComp
 $Comp
-L +3.3V #PWR017
+L +3.3V #PWR021
 U 1 1 4D9FC667
 P 4050 6150
-F 0 "#PWR017" H 4050 6110 30  0001 C CNN
+F 0 "#PWR021" H 4050 6110 30  0001 C CNN
 F 1 "+3.3V" H 4050 6260 30  0000 C CNN
 	1    4050 6150
@@
 $EndComp
 $Comp
-L +3.3V #PWR018
+L +3.3V #PWR022
 U 1 1 4D9FC639
 P 1600 4450
-F 0 "#PWR018" H 1600 4410 30  0001 C CNN
+F 0 "#PWR022" H 1600 4410 30  0001 C CNN
 F 1 "+3.3V" H 1600 4560 30  0000 C CNN
 	1    1600 4450
@@
 $EndComp
 $Comp
-L GND #PWR019
+L GND #PWR023
 U 1 1 4D9FC633
 P 2700 5000
-F 0 "#PWR019" H 2700 5000 30  0001 C CNN
+F 0 "#PWR023" H 2700 5000 30  0001 C CNN
 F 1 "GND" H 2700 4930 30  0001 C CNN
 	1    2700 5000
@@
 $EndComp
 $Comp
-L GND #PWR020
+L GND #PWR024
 U 1 1 4D9FBFA4
 P 5600 6900
-F 0 "#PWR020" H 5600 6900 30  0001 C CNN
+F 0 "#PWR024" H 5600 6900 30  0001 C CNN
 F 1 "GND" H 5600 6830 30  0001 C CNN
 	1    5600 6900
@@
 $EndComp
 $Comp
-L +3.3V #PWR021
+L +3.3V #PWR025
 U 1 1 4D9FBF87
 P 2600 2800
-F 0 "#PWR021" H 2600 2760 30  0001 C CNN
+F 0 "#PWR025" H 2600 2760 30  0001 C CNN
 F 1 "+3.3V" H 2600 2910 30  0000 C CNN
 	1    2600 2800
@@
 $EndComp
 $Comp
-L GND #PWR022
+L GND #PWR026
 U 1 1 4D9FBF37
 P 1800 3100
-F 0 "#PWR022" H 1800 3100 30  0001 C CNN
+F 0 "#PWR026" H 1800 3100 30  0001 C CNN
 F 1 "GND" H 1800 3030 30  0001 C CNN
 	1    1800 3100
@@
 $EndComp
 $Comp
-L GND #PWR023
+L GND #PWR027
 U 1 1 4D9FBEF0
 P 3500 1800
-F 0 "#PWR023" H 3500 1800 30  0001 C CNN
+F 0 "#PWR027" H 3500 1800 30  0001 C CNN
 F 1 "GND" H 3500 1730 30  0001 C CNN
 	1    3500 1800
@@
 $EndComp
 $Comp
-L GND #PWR024
+L GND #PWR028
 U 1 1 4D9FBBA7
 P 6900 2050
-F 0 "#PWR024" H 6900 2050 30  0001 C CNN
+F 0 "#PWR028" H 6900 2050 30  0001 C CNN
 F 1 "GND" H 6900 1980 30  0001 C CNN
 	1    6900 2050
@@
 $EndComp
 $Comp
-L +3.3V #PWR025
+L +3.3V #PWR029
 U 1 1 4D9FBB67
 P 5600 1300
-F 0 "#PWR025" H 5600 1260 30  0001 C CNN
+F 0 "#PWR029" H 5600 1260 30  0001 C CNN
 F 1 "+3.3V" H 5600 1410 30  0000 C CNN
 	1    5600 1300
@@
 $EndComp
 $Comp
-L GND #PWR026
+L GND #PWR030
 U 1 1 4D9FBB51
 P 5050 1750
-F 0 "#PWR026" H 5050 1750 30  0001 C CNN
+F 0 "#PWR030" H 5050 1750 30  0001 C CNN
 F 1 "GND" H 5050 1680 30  0001 C CNN
 	1    5050 1750

Commit message: Reruteo a 10mils/9.6mils en placas LPC1754 y STM32F105R8T6
Parts:
- removed JP2: JUMPER-3, symbol JUMPER-3
- added J2: PWR_SELF, symbol JUMPER-2
- added J3: PWR_USB, symbol JUMPER-2
- J1: renamed from JPRG1; value JUMPER-2 -> ISP
- J4: renamed from J_HOST1; value USB_2 -> USB_HOST
- J5: renamed from J1; value USB -> USB_DEV
Connections:
- net labels added: PWR, PWR_SELF
- net labels removed: +5V
- wire segments 181 -> 182
